File: frontend/BPF Superband/basic-superband-pa.kicad_pcb (KiCad board)
At the start: 2 copper layers, 64.5 x 60 mm, 81 parts, among them CN1 EDGE, K1 D3002, K2 D3002, P1 BNC, P2 VFWD, P3 Ext PTT, P4 12-13.8v, Q1 FDV301, Q2 FDV301, Q3 RD16HHF1, T2 8:1, T3 4:1, T4 OUT_TRANSF, U1 LP2951-50D

Commit message: New pre-v2 files
Parts:
- removed C32: 0.1uF, HERMESLITE:C_0805
Connections:
- P2 pad 2: Net-(C32-Pad1) -> Net-(P2-Pad2)
- R10 pad 2: Net-(C32-Pad1) -> Net-(P2-Pad2)
- R11 pad 2: Net-(C32-Pad1) -> Net-(P2-Pad2)
- T3 pad 1: Net-(C32-Pad2) -> Net-(P2-Pad2)
Routing:
- net Net-(C32-Pad1): track 12.9 -> 0.00 mm
- net Net-(P2-Pad2): track 0.00 -> 11.8 mm
- net Net-(C32-Pad2): track 4.06 -> 0.00 mm
