File: frontend/BPF Superband/basic-superband-pa.sch (KiCad schematic (older format))
At the start: 76 parts, among them CN1 EDGE, K1 D3002, K2 D3002, P1 BNC, P2 VFWD, P3 Ext PTT, P4 12-13.8v, Q1 FDV301, Q2 FDV301, Q3 RD16HHF1, T2 8:1, T3 4:1, T4 OUT_TRANSF, U1 LP2951-50D

Commit message: New pre-v2 files
Parts:
- removed C32: 0.1uF, HERMESLITE:C_0805, symbol C
Connections:
- net at T3.1 (S1): now also P2.2 (P2), R10.2, R11.2
Other:
- note added: "4T bifilar\n6T\nBN-43-2402"
- note added: "6T bifilar\n4T\nBN-43-2402"
- note removed: "4T bifilar\n6T\nBN-61-2402"
- note removed: "6T bifilar\n4T\nBN-61-2402"
- moved on the sheet: P2
Changed lines of the file:
@@
 $EndComp
 Text Notes 4000 3600 0    60   ~ 0
-6T bifilar\n4T\nBN-61-2402
+6T bifilar\n4T\nBN-43-2402
 Text Notes 4500 3050 0    60   ~ 0
-4T bifilar\n6T\nBN-61-2402
+4T bifilar\n6T\nBN-43-2402
 $Comp
 L C C15
@@
 L CONN_02X01 P2
 U 1 1 554E215A
-P 5500 2550
-F 0 "P2" V 5500 2450 50  0000 C CNN
-F 1 "VFWD" H 5500 2650 50  0000 C CNN
-F 2 "Pin_Headers:Pin_Header_Straight_1x02" H 5500 1350 60  0001 C CNN
-F 3 "" H 5500 1350 60  0000 C CNN
-	1    5500 2550
+P 5400 2500
+F 0 "P2" V 5400 2400 50  0000 C CNN
+F 1 "VFWD" H 5400 2600 50  0000 C CNN
+F 2 "Pin_Headers:Pin_Header_Straight_1x02" H 5400 1300 60  0001 C CNN
+F 3 "" H 5400 1300 60  0000 C CNN
+	1    5400 2500
 	0    -1   -1   0
 $EndComp
@@
 Connection ~ 6350 2350
 Connection ~ 8650 1150
-$Comp
-L C C32
-U 1 1 554E53AA
-P 5400 2200
-F 0 "C32" V 5300 2000 40  0000 L CNN
-F 1 "0.1uF" V 5500 1950 40  0000 L CNN
-F 2 "HERMESLITE:C_0805" H 5438 2050 30  0001 C CNN
-F 3 "" H 5400 2200 60  0000 C CNN
-	1    5400 2200
-	0    1    1    0
-$EndComp
 Wire Wire Line
 	6250 2950 6250 2200
@@
 	6250 2200 6150 2200
 Wire Wire Line
-	5600 2200 5650 2200
-Wire Wire Line
-	5600 2200 5600 2250
-Wire Wire Line
-	5600 2250 5550 2250
-Wire Wire Line
-	5550 2250 5550 2300
-Wire Wire Line
-	5550 2300 5500 2300
+	5200 2200 5650 2200
 Wire Wire Line
 	5200 2600 5200 2800
@@
 Wire Wire Line
 	5650 2800 5650 2700
-Connection ~ 5500 2800
 Wire Wire Line
 	5800 2800 5800 2700
@@
 Connection ~ 4700 7350
 Connection ~ 4700 7750
+Wire Wire Line
+	5400 2750 5400 2800
+Connection ~ 5400 2800
+Wire Wire Line
+	5400 2250 5400 2200
+Connection ~ 5400 2200
 $EndSCHEMATC
