File: interface/waveshare/waveshare.kicad_pcb (KiCad board)
At the start: 2 copper layers, 25.2 x 17.9 mm, 2 parts, among them CN1 WaveShare Angle, CN2 WaveShare Edge

Commit message: Latest Rx updates
Parts:
- moved CN2 16.5 mm to (152.7, 105.5), turned to 90 degrees
Routing:
- net Net-(CN1-Pad1): track 65.1 -> 22.5 mm
- net Net-(CN1-Pad11): track 8.16 -> 32.8 mm
- net Net-(CN1-Pad9): track 16.2 -> 29.2 mm
- net Net-(CN1-Pad10): track 14.5 -> 26.6 mm
- net Net-(CN1-Pad2): track 61.4 -> 49.3 mm
- net Net-(CN1-Pad7): track 18.6 -> 26.7 mm
- net Net-(CN1-Pad8): track 16.4 -> 22.9 mm
- net Net-(CN1-Pad5): track 20.7 -> 24.2 mm
- net Net-(CN1-Pad4): track 20.8 -> 18.8 mm
- net Net-(CN1-Pad6): track 18.1 -> 20.1 mm
- net Net-(CN1-Pad3): track 24.5 -> 23.0 mm
Other:
- board size 25.2 x 17.9 mm -> 27.9 x 17.9 mm
