File: frontend/v2-Amp/amp.kicad_pcb (KiCad board)
At the start: 4 copper layers, 80 x 100 mm, 154 parts, among them K1 HK4100, K10 HK4100, K11 HK4100, K12 HK4100, K13 HK4100, K14 HK4100, K15 HK4100, K2 HK4100, K3 HK4100, K4 HK4100, K5 HK4100, K6 HK4100, K7 HK4100, K8 HK4100, K9 HK4100, P1 Antenna, P2 CONN_02X07, P3 TX Power Tap, P4 TX-IN, P5 RX IN, P6 12-13.8v, Q2 RD16HHF1, T1 OUT_TRANSF, U1 LP2951-50D

Commit message: Updates for v1.1
Parts:
- added C63: DNI, HERMESLITE:C_0805, B.Cu at (165.2, 124.3)
- added C64: 100pf, HERMESLITE:C_0805, B.Cu at (172.9, 125.7)
- added L22: 330nH, HERMESLITE:inductor, F.Cu at (168.0, 126.2)
- C11, C8, C9, R15, R16, R17: moved to F.Cu
- C21, C22, C23, C24, C25, C26, C27, C28, C29, C30, C31, C32, C33, C34, C35, C36, C37, C38, C39, C40, C41, C42, C43, C44, C45, C46, C47, C48, C49, C50, C51, C52, C53, C54, C55, C56, C57, C58, C59, C60, C61, C62: moved to B.Cu
- moved C2 11.9 mm to (150.1, 125.7), turned to 270 degrees
- moved C6 6.12 mm to (172.0, 128.3)
- moved C3 5.28 mm to (161.3, 126.6)
- moved C4 4.24 mm to (152.7, 127.7), turned to 90 degrees
- moved L2 4.20 mm to (162.6, 128.8), turned to 90 degrees
- moved C28 3.37 mm to (157.2, 72.9), turned to 90 degrees
- moved L1 3.33 mm to (157.2, 126.2)
- moved C27 3.13 mm to (157.3, 62.2), turned to 90 degrees
- moved C29 3.12 mm to (157.2, 84.0), turned to 90 degrees
- moved C31 3.00 mm to (157.2, 105.7), turned to 90 degrees
- moved C32 2.98 mm to (157.3, 116.5), turned to 90 degrees
- moved C30 2.48 mm to (157.6, 94.8), turned to 90 degrees
- moved C11 2.18 mm to (119.7, 71.3), turned to 0 degrees
- moved C5 1.55 mm to (165.7, 130.6)
- moved C51 1.44 mm to (173.3, 62.0), turned to 90 degrees
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Connections:
- K15 pad 4: Net-(C5-Pad1) -> Net-(C63-Pad1)
Routing:
- net Net-(C63-Pad1): track 0.00 -> 15.9 mm
- net Net-(C11-Pad2): track 24.6 -> 15.7 mm, vias 0 -> 1
- net +12v: track 351.9 -> 357.7 mm
- net GND: track 183.7 -> 187.4 mm, vias 38 -> 39
- net Net-(C2-Pad1): track 15.3 -> 12.5 mm
- net Net-(C5-Pad1): track 14.5 -> 16.8 mm
- net /PTT: track 132.8 -> 130.5 mm
- net Net-(C9-Pad2): track 19.8 -> 21.7 mm
- net Net-(C42-Pad1): track 11.7 -> 13.6 mm
- net Net-(C3-Pad1): track 19.1 -> 18.1 mm
- net Net-(C31-Pad1): track 12.7 -> 13.7 mm
- net /Band1: track 113.4 -> 112.5 mm
- net /Band5: track 77.8 -> 77.1 mm
- net /Band4: track 90.6 -> 89.8 mm
- net /Band2: track 102.0 -> 101.2 mm
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Other:
- board text added: "Hermes Lite Pre-V2 PA 1.1 © 2016 W9JSW"
- board text removed: "Hermes Lite Pre-V2 PA 1.2 © 2016 W9JSW"

Commit message: bom change
Parts:
- moved C17 2.84 mm to (131.7, 54.2)
- moved C18 2.77 mm to (128.5, 54.2)
- moved C16 2.68 mm to (125.5, 54.2)
- moved C19 2.67 mm to (122.3, 54.2)
Routing:
- net GND: track 187.4 -> 164.0 mm, vias 39 -> 45
- net Net-(C16-Pad2): track 41.4 -> 36.2 mm
- net /Band2: track 101.2 -> 100.5 mm
